File: PCB´s/VoltimetroTrifasico/sch.brd (EAGLE design)
At the start: 160 x 100 mm, 22 parts, among them IC1 LM324N

Commit message: probando 2
Parts:
- moved IC1 126.9 mm to (52.1, 85.1)
- moved R3 87.7 mm to (15.2, 43.2)
- moved R2 80.7 mm to (15.2, 31.8)
- moved R11 37.6 mm to (12.7, 52.1)
Changed lines of the file:
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@@
 <attribute name="MF" value="" x="60.96" y="29.21" size="1.778" layer="27" display="off"/>
 </element>
-<element name="IC1" library="linear" package="DIL14" value="LM324N" x="-68.58" y="45.72"/>
+<element name="IC1" library="linear" package="DIL14" value="LM324N" x="52.07" y="85.09"/>
 <element name="R1" library="rcl" package="0204/7" value="10k" x="-50.8" y="58.42"/>
 <element name="R10" library="rcl" package="0204/7" value="10k" x="-68.58" y="66.04"/>
-<element name="R11" library="pot" package="B64Y" value="" x="-24.13" y="59.69"/>
+<element name="R11" library="pot" package="B64Y" value="" x="12.7" y="52.07"/>
 <element name="R12" library="rcl" package="0204/7" value="10k" x="-78.74" y="66.04"/>
 <element name="R13" library="rcl" package="0204/7" value="100k" x="-17.78" y="69.85"/>
@@
 <element name="R17" library="rcl" package="0204/7" value="10k" x="-48.26" y="69.85"/>
 <element name="R18" library="rcl" package="0204/7" value="10k" x="-58.42" y="69.85"/>
-<element name="R2" library="rcl" package="0204/7" value="100k" x="-60.96" y="58.42"/>
-<element name="R3" library="rcl" package="0204/7" value="10k" x="-71.12" y="58.42"/>
+<element name="R2" library="rcl" package="0204/7" value="100k" x="15.24" y="31.75"/>
+<element name="R3" library="rcl" package="0204/7" value="10k" x="15.24" y="43.18"/>
 <element name="R4" library="rcl" package="0204/7" value="10k" x="-17.78" y="66.04"/>
 <element name="R5" library="rcl" package="0204/7" value="10k" x="-27.94" y="66.04"/>
@@
 <contactref element="R5" pad="2"/>
 <contactref element="IC1" pad="2"/>
-<wire x1="-73.66" y1="41.91" x2="-24.13" y2="66.04" width="0" layer="19" extent="1-1"/>
+<wire x1="46.99" y1="81.28" x2="-24.13" y2="66.04" width="0" layer="19" extent="1-1"/>
 </signal>
 <signal name="IN1">
@@
 <contactref element="R2" pad="2"/>
 <wire x1="-54.61" y1="58.42" x2="-21.59" y2="66.04" width="0" layer="19" extent="1-1"/>
-<wire x1="-57.15" y1="58.42" x2="-54.61" y2="58.42" width="0" layer="19" extent="1-1"/>
-<wire x1="-74.93" y1="58.42" x2="-57.15" y2="58.42" width="0" layer="19" extent="1-1"/>
-<wire x1="-71.12" y1="41.91" x2="-74.93" y2="58.42" width="0" layer="19" extent="1-1"/>
+<wire x1="19.05" y1="31.75" x2="-54.61" y2="58.42" width="0" layer="19" extent="1-1"/>
+<wire x1="11.43" y1="43.18" x2="19.05" y2="31.75" width="0" layer="19" extent="1-1"/>
+<wire x1="49.53" y1="81.28" x2="11.43" y2="43.18" width="0" layer="19" extent="1-1"/>
 </signal>
 <signal name="OFFSET1">
@@
 <contactref element="220" pad="2"/>
 <wire x1="39.12" y1="44.71" x2="28.96" y2="44.71" width="0" layer="19" extent="1-1"/>
-<wire x1="-68.58" y1="49.53" x2="39.12" y2="44.71" width="0" layer="19" extent="1-1"/>
-<wire x1="-67.31" y1="58.42" x2="-68.58" y2="49.53" width="0" layer="19" extent="1-1"/>
-<wire x1="-36.83" y1="58.42" x2="-67.31" y2="58.42" width="0" layer="19" extent="1-1"/>
+<wire x1="52.07" y1="88.9" x2="39.12" y2="44.71" width="0" layer="19" extent="1-1"/>
+<wire x1="19.05" y1="43.18" x2="52.07" y2="88.9" width="0" layer="19" extent="1-1"/>
+<wire x1="-36.83" y1="58.42" x2="19.05" y2="43.18" width="0" layer="19" extent="1-1"/>
 <wire x1="-29.21" y1="59.69" x2="-36.83" y2="58.42" width="0" layer="19" extent="1-1"/>
 <wire x1="45.72" y1="73.66" x2="-29.21" y2="59.69" width="0" layer="19" extent="1-1"/>
@@
 <contactref element="DIS1" pad="2"/>
 <contactref element="DIS1" pad="15"/>
-<wire x1="-68.58" y1="41.91" x2="31.5" y2="44.71" width="0" layer="19" extent="1-1"/>
-<wire x1="64.52" y1="44.71" x2="-68.58" y2="41.91" width="0" layer="19" extent="1-1"/>
+<wire x1="52.07" y1="81.28" x2="31.5" y2="44.71" width="0" layer="19" extent="1-1"/>
+<wire x1="64.52" y1="44.71" x2="52.07" y2="81.28" width="0" layer="19" extent="1-1"/>
 <wire x1="-34.29" y1="59.69" x2="64.52" y2="44.71" width="0" layer="19" extent="1-1"/>
 <wire x1="-19.05" y1="59.69" x2="-34.29" y2="59.69" width="0" layer="19" extent="1-1"/>
@@
 <contactref element="R7" pad="1"/>
 <contactref element="R8" pad="2"/>
-<wire x1="-62.23" y1="66.04" x2="-66.04" y2="41.91" width="0" layer="19" extent="1-1"/>
+<wire x1="-62.23" y1="66.04" x2="54.61" y2="81.28" width="0" layer="19" extent="1-1"/>
 <wire x1="-72.39" y1="66.04" x2="-62.23" y2="66.04" width="0" layer="19" extent="1-1"/>
 <wire x1="-44.45" y1="66.04" x2="-62.23" y2="66.04" width="0" layer="19" extent="1-1"/>
@@
 <contactref element="R10" pad="2"/>
 <contactref element="R11" pad="S"/>
-<wire x1="-64.77" y1="66.04" x2="-24.13" y2="59.69" width="0" layer="19" extent="1-1"/>
+<wire x1="-64.77" y1="66.04" x2="12.7" y2="52.07" width="0" layer="19" extent="1-1"/>
 </signal>
 <signal name="GND1">
 <contactref element="R9" pad="2"/>
 <contactref element="R11" pad="A"/>
-<wire x1="-54.61" y1="66.04" x2="-21.59" y2="59.69" width="0" layer="19" extent="1-1"/>
+<wire x1="-54.61" y1="66.04" x2="15.24" y2="52.07" width="0" layer="19" extent="1-1"/>
 </signal>
 <signal name="+5V1">
@@
 <wire x1="-31.75" y1="69.85" x2="-13.97" y2="69.85" width="0" layer="19" extent="1-1"/>
 <wire x1="-41.91" y1="69.85" x2="-31.75" y2="69.85" width="0" layer="19" extent="1-1"/>
-<wire x1="-66.04" y1="49.53" x2="-41.91" y2="69.85" width="0" layer="19" extent="1-1"/>
-<wire x1="-82.55" y1="66.04" x2="-66.04" y2="49.53" width="0" layer="19" extent="1-1"/>
+<wire x1="54.61" y1="88.9" x2="-41.91" y2="69.85" width="0" layer="19" extent="1-1"/>
+<wire x1="-82.55" y1="66.04" x2="54.61" y2="88.9" width="0" layer="19" extent="1-1"/>
 </signal>
 <signal name="OFFSET3">
@@
 <contactref element="R18" pad="2"/>
 <contactref element="IC1" pad="9"/>
-<wire x1="-63.5" y1="49.53" x2="-54.61" y2="69.85" width="0" layer="19" extent="1-1"/>
+<wire x1="57.15" y1="88.9" x2="-54.61" y2="69.85" width="0" layer="19" extent="1-1"/>
 </signal>
 <signal name="N$5">
 <contactref element="R17" pad="2"/>
 <contactref element="IC1" pad="6"/>
-<wire x1="-63.5" y1="41.91" x2="-44.45" y2="69.85" width="0" layer="19" extent="1-1"/>
+<wire x1="57.15" y1="81.28" x2="-44.45" y2="69.85" width="0" layer="19" extent="1-1"/>
 </signal>
 <signal name="AN0">
@@
 <contactref element="IC1" pad="1"/>
 <wire x1="25.4" y1="58.42" x2="-31.75" y2="66.04" width="0" layer="19" extent="1-1"/>
-<wire x1="-76.2" y1="41.91" x2="25.4" y2="58.42" width="0" layer="19" extent="1-1"/>
+<wire x1="44.45" y1="81.28" x2="25.4" y2="58.42" width="0" layer="19" extent="1-1"/>
 </signal>
 <signal name="AN1">
@@
 <contactref element="R17" pad="1"/>
 <contactref element="IC1" pad="7"/>
-<wire x1="27.94" y1="58.42" x2="-60.96" y2="41.91" width="0" layer="19" extent="1-1"/>
-<wire x1="-52.07" y1="69.85" x2="-60.96" y2="41.91" width="0" layer="19" extent="1-1"/>
+<wire x1="27.94" y1="58.42" x2="59.69" y2="81.28" width="0" layer="19" extent="1-1"/>
+<wire x1="-52.07" y1="69.85" x2="59.69" y2="81.28" width="0" layer="19" extent="1-1"/>
 </signal>
 <signal name="AN2">
@@
 <contactref element="R18" pad="1"/>
 <contactref element="IC1" pad="8"/>
-<wire x1="-62.23" y1="69.85" x2="-60.96" y2="49.53" width="0" layer="19" extent="1-1"/>
-<wire x1="30.48" y1="58.42" x2="-60.96" y2="49.53" width="0" layer="19" extent="1-1"/>
+<wire x1="-62.23" y1="69.85" x2="59.69" y2="88.9" width="0" layer="19" extent="1-1"/>
+<wire x1="30.48" y1="58.42" x2="59.69" y2="88.9" width="0" layer="19" extent="1-1"/>
 </signal>
 <signal name="N$13">
