File: PCB´s/VoltimetroTrifasico/sch2.brd (EAGLE design)
At the start: 160 x 100 mm, 22 parts, among them IC1 LM324N

Commit message: movi lcd
Parts:
- moved ARDUINO_NANO1 88.7 mm to (125.7, 25.4)
- moved DIS1 20.5 mm to (95.2, 58.4)
Changed lines of the file:
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@@
 <elements>
 <element name="220" library="rcl" package="0204/7" value="10k" x="-40.64" y="58.42"/>
-<element name="ARDUINO_NANO1" library="ArduinoNanoV30" package="ARDUINO_NANO" value="" x="38.1" y="39.37"/>
-<element name="DIS1" library="display-lcd" package="TUXGR_16X2_R2" value="TUXGR_16X2_R2" x="114.3" y="66.04">
-<attribute name="MPN" value="" x="114.3" y="66.04" size="1.778" layer="27" display="off"/>
-<attribute name="OC_FARNELL" value="unknown" x="114.3" y="66.04" size="1.778" layer="27" display="off"/>
-<attribute name="OC_NEWARK" value="unknown" x="114.3" y="66.04" size="1.778" layer="27" display="off"/>
-<attribute name="MF" value="" x="114.3" y="66.04" size="1.778" layer="27" display="off"/>
+<element name="ARDUINO_NANO1" library="ArduinoNanoV30" package="ARDUINO_NANO" value="" x="125.73" y="25.4"/>
+<element name="DIS1" library="display-lcd" package="TUXGR_16X2_R2" value="TUXGR_16X2_R2" x="95.25" y="58.42">
+<attribute name="MPN" value="" x="95.25" y="58.42" size="1.778" layer="27" display="off"/>
+<attribute name="OC_FARNELL" value="unknown" x="95.25" y="58.42" size="1.778" layer="27" display="off"/>
+<attribute name="OC_NEWARK" value="unknown" x="95.25" y="58.42" size="1.778" layer="27" display="off"/>
+<attribute name="MF" value="" x="95.25" y="58.42" size="1.778" layer="27" display="off"/>
 </element>
 <element name="IC1" library="linear" package="DIL14" value="LM324N" x="52.07" y="85.09"/>
@@
 <contactref element="DIS1" pad="5"/>
 <contactref element="220" pad="2"/>
-<wire x1="92.46" y1="81.54" x2="82.3" y2="81.54" width="0" layer="19" extent="1-1"/>
-<wire x1="52.07" y1="88.9" x2="92.46" y2="81.54" width="0" layer="19" extent="1-1"/>
+<wire x1="73.41" y1="73.92" x2="63.25" y2="73.92" width="0" layer="19" extent="1-1"/>
+<wire x1="52.07" y1="88.9" x2="73.41" y2="73.92" width="0" layer="19" extent="1-1"/>
 <wire x1="19.05" y1="43.18" x2="52.07" y2="88.9" width="0" layer="19" extent="1-1"/>
 <wire x1="-36.83" y1="58.42" x2="19.05" y2="43.18" width="0" layer="19" extent="1-1"/>
 <wire x1="-29.21" y1="59.69" x2="-36.83" y2="58.42" width="0" layer="19" extent="1-1"/>
-<wire x1="45.72" y1="46.99" x2="-29.21" y2="59.69" width="0" layer="19" extent="1-1"/>
+<wire x1="133.35" y1="33.02" x2="-29.21" y2="59.69" width="0" layer="19" extent="1-1"/>
 <wire x1="-24.13" y1="69.85" x2="-29.21" y2="59.69" width="0" layer="19" extent="1-1"/>
-<wire x1="-13.97" y1="59.69" x2="45.72" y2="46.99" width="0" layer="19" extent="1-1"/>
-<wire x1="50.8" y1="31.75" x2="45.72" y2="46.99" width="0" layer="19" extent="1-1"/>
+<wire x1="-13.97" y1="59.69" x2="133.35" y2="33.02" width="0" layer="19" extent="1-1"/>
+<wire x1="138.43" y1="17.78" x2="133.35" y2="33.02" width="0" layer="19" extent="1-1"/>
 </signal>
 <signal name="+5V">
@@
 <contactref element="DIS1" pad="2"/>
 <contactref element="DIS1" pad="15"/>
-<wire x1="52.07" y1="81.28" x2="84.84" y2="81.54" width="0" layer="19" extent="1-1"/>
-<wire x1="117.86" y1="81.54" x2="52.07" y2="81.28" width="0" layer="19" extent="1-1"/>
-<wire x1="-34.29" y1="59.69" x2="117.86" y2="81.54" width="0" layer="19" extent="1-1"/>
+<wire x1="52.07" y1="81.28" x2="65.79" y2="73.92" width="0" layer="19" extent="1-1"/>
+<wire x1="98.81" y1="73.92" x2="52.07" y2="81.28" width="0" layer="19" extent="1-1"/>
+<wire x1="-34.29" y1="59.69" x2="98.81" y2="73.92" width="0" layer="19" extent="1-1"/>
 <wire x1="-19.05" y1="59.69" x2="-34.29" y2="59.69" width="0" layer="19" extent="1-1"/>
-<wire x1="53.34" y1="31.75" x2="-19.05" y2="59.69" width="0" layer="19" extent="1-1"/>
+<wire x1="140.97" y1="17.78" x2="-19.05" y2="59.69" width="0" layer="19" extent="1-1"/>
 </signal>
 <signal name="AC1_3">
@@
 <contactref element="R5" pad="1"/>
 <contactref element="IC1" pad="1"/>
-<wire x1="25.4" y1="31.75" x2="-31.75" y2="66.04" width="0" layer="19" extent="1-1"/>
-<wire x1="44.45" y1="81.28" x2="25.4" y2="31.75" width="0" layer="19" extent="1-1"/>
+<wire x1="113.03" y1="17.78" x2="-31.75" y2="66.04" width="0" layer="19" extent="1-1"/>
+<wire x1="44.45" y1="81.28" x2="113.03" y2="17.78" width="0" layer="19" extent="1-1"/>
 </signal>
 <signal name="AN1">
@@
 <contactref element="R17" pad="1"/>
 <contactref element="IC1" pad="7"/>
-<wire x1="27.94" y1="31.75" x2="59.69" y2="81.28" width="0" layer="19" extent="1-1"/>
+<wire x1="115.57" y1="17.78" x2="59.69" y2="81.28" width="0" layer="19" extent="1-1"/>
 <wire x1="-52.07" y1="69.85" x2="59.69" y2="81.28" width="0" layer="19" extent="1-1"/>
 </signal>
@@
 <contactref element="IC1" pad="8"/>
 <wire x1="-62.23" y1="69.85" x2="59.69" y2="88.9" width="0" layer="19" extent="1-1"/>
-<wire x1="30.48" y1="31.75" x2="59.69" y2="88.9" width="0" layer="19" extent="1-1"/>
+<wire x1="118.11" y1="17.78" x2="59.69" y2="88.9" width="0" layer="19" extent="1-1"/>
 </signal>
 <signal name="N$13">
@@
 <contactref element="ARDUINO_NANO1" pad="26"/>
 <contactref element="DIS1" pad="11"/>
-<wire x1="27.94" y1="46.99" x2="107.7" y2="81.54" width="0" layer="19" extent="1-1"/>
+<wire x1="115.57" y1="33.02" x2="88.65" y2="73.92" width="0" layer="19" extent="1-1"/>
 </signal>
 <signal name="D7">
 <contactref element="ARDUINO_NANO1" pad="22"/>
 <contactref element="DIS1" pad="14"/>
-<wire x1="115.32" y1="81.54" x2="38.1" y2="46.99" width="0" layer="19" extent="1-1"/>
+<wire x1="96.27" y1="73.92" x2="125.73" y2="33.02" width="0" layer="19" extent="1-1"/>
 </signal>
 <signal name="D6">
 <contactref element="ARDUINO_NANO1" pad="23"/>
 <contactref element="DIS1" pad="13"/>
-<wire x1="112.78" y1="81.54" x2="35.56" y2="46.99" width="0" layer="19" extent="1-1"/>
+<wire x1="93.73" y1="73.92" x2="123.19" y2="33.02" width="0" layer="19" extent="1-1"/>
 </signal>
 <signal name="D5">
 <contactref element="ARDUINO_NANO1" pad="24"/>
 <contactref element="DIS1" pad="12"/>
-<wire x1="33.02" y1="46.99" x2="110.24" y2="81.54" width="0" layer="19" extent="1-1"/>
+<wire x1="120.65" y1="33.02" x2="91.19" y2="73.92" width="0" layer="19" extent="1-1"/>
 </signal>
 <signal name="ENA">
 <contactref element="ARDUINO_NANO1" pad="28"/>
 <contactref element="DIS1" pad="6"/>
-<wire x1="22.86" y1="46.99" x2="95" y2="81.54" width="0" layer="19" extent="1-1"/>
+<wire x1="110.49" y1="33.02" x2="75.95" y2="73.92" width="0" layer="19" extent="1-1"/>
 </signal>
 <signal name="RS">
 <contactref element="ARDUINO_NANO1" pad="29"/>
 <contactref element="DIS1" pad="4"/>
-<wire x1="20.32" y1="46.99" x2="89.92" y2="81.54" width="0" layer="19" extent="1-1"/>
+<wire x1="107.95" y1="33.02" x2="70.87" y2="73.92" width="0" layer="19" extent="1-1"/>
 </signal>
 <signal name="V0">
@@
 <contactref element="DIS1" pad="16"/>
 <contactref element="220" pad="1"/>
-<wire x1="120.4" y1="81.54" x2="-44.45" y2="58.42" width="0" layer="19" extent="1-1"/>
+<wire x1="101.35" y1="73.92" x2="-44.45" y2="58.42" width="0" layer="19" extent="1-1"/>
 </signal>
 </signals>

Commit message: movi
Parts:
- moved IC1 36.9 mm to (88.9, 87.6)
Changed lines of the file:
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@@
 <attribute name="MF" value="" x="95.25" y="58.42" size="1.778" layer="27" display="off"/>
 </element>
-<element name="IC1" library="linear" package="DIL14" value="LM324N" x="52.07" y="85.09"/>
+<element name="IC1" library="linear" package="DIL14" value="LM324N" x="88.9" y="87.63"/>
 <element name="R1" library="rcl" package="0204/7" value="10k" x="-50.8" y="58.42"/>
 <element name="R10" library="rcl" package="0204/7" value="10k" x="-68.58" y="66.04"/>
@@
 <contactref element="R5" pad="2"/>
 <contactref element="IC1" pad="2"/>
-<wire x1="46.99" y1="81.28" x2="-24.13" y2="66.04" width="0" layer="19" extent="1-1"/>
+<wire x1="83.82" y1="83.82" x2="-24.13" y2="66.04" width="0" layer="19" extent="1-1"/>
 </signal>
 <signal name="IN1">
@@
 <wire x1="19.05" y1="31.75" x2="-54.61" y2="58.42" width="0" layer="19" extent="1-1"/>
 <wire x1="11.43" y1="43.18" x2="19.05" y2="31.75" width="0" layer="19" extent="1-1"/>
-<wire x1="49.53" y1="81.28" x2="11.43" y2="43.18" width="0" layer="19" extent="1-1"/>
+<wire x1="86.36" y1="83.82" x2="11.43" y2="43.18" width="0" layer="19" extent="1-1"/>
 </signal>
 <signal name="OFFSET1">
@@
 <contactref element="220" pad="2"/>
 <wire x1="73.41" y1="73.92" x2="63.25" y2="73.92" width="0" layer="19" extent="1-1"/>
-<wire x1="52.07" y1="88.9" x2="73.41" y2="73.92" width="0" layer="19" extent="1-1"/>
-<wire x1="19.05" y1="43.18" x2="52.07" y2="88.9" width="0" layer="19" extent="1-1"/>
+<wire x1="88.9" y1="91.44" x2="73.41" y2="73.92" width="0" layer="19" extent="1-1"/>
+<wire x1="19.05" y1="43.18" x2="88.9" y2="91.44" width="0" layer="19" extent="1-1"/>
 <wire x1="-36.83" y1="58.42" x2="19.05" y2="43.18" width="0" layer="19" extent="1-1"/>
 <wire x1="-29.21" y1="59.69" x2="-36.83" y2="58.42" width="0" layer="19" extent="1-1"/>
@@
 <contactref element="DIS1" pad="2"/>
 <contactref element="DIS1" pad="15"/>
-<wire x1="52.07" y1="81.28" x2="65.79" y2="73.92" width="0" layer="19" extent="1-1"/>
-<wire x1="98.81" y1="73.92" x2="52.07" y2="81.28" width="0" layer="19" extent="1-1"/>
+<wire x1="88.9" y1="83.82" x2="65.79" y2="73.92" width="0" layer="19" extent="1-1"/>
+<wire x1="98.81" y1="73.92" x2="88.9" y2="83.82" width="0" layer="19" extent="1-1"/>
 <wire x1="-34.29" y1="59.69" x2="98.81" y2="73.92" width="0" layer="19" extent="1-1"/>
 <wire x1="-19.05" y1="59.69" x2="-34.29" y2="59.69" width="0" layer="19" extent="1-1"/>
@@
 <contactref element="R7" pad="1"/>
 <contactref element="R8" pad="2"/>
-<wire x1="-62.23" y1="66.04" x2="54.61" y2="81.28" width="0" layer="19" extent="1-1"/>
+<wire x1="-62.23" y1="66.04" x2="91.44" y2="83.82" width="0" layer="19" extent="1-1"/>
 <wire x1="-72.39" y1="66.04" x2="-62.23" y2="66.04" width="0" layer="19" extent="1-1"/>
 <wire x1="-44.45" y1="66.04" x2="-62.23" y2="66.04" width="0" layer="19" extent="1-1"/>
@@
 <wire x1="-31.75" y1="69.85" x2="-13.97" y2="69.85" width="0" layer="19" extent="1-1"/>
 <wire x1="-41.91" y1="69.85" x2="-31.75" y2="69.85" width="0" layer="19" extent="1-1"/>
-<wire x1="54.61" y1="88.9" x2="-41.91" y2="69.85" width="0" layer="19" extent="1-1"/>
-<wire x1="-82.55" y1="66.04" x2="54.61" y2="88.9" width="0" layer="19" extent="1-1"/>
+<wire x1="91.44" y1="91.44" x2="-41.91" y2="69.85" width="0" layer="19" extent="1-1"/>
+<wire x1="-82.55" y1="66.04" x2="91.44" y2="91.44" width="0" layer="19" extent="1-1"/>
 </signal>
 <signal name="OFFSET3">
@@
 <contactref element="R18" pad="2"/>
 <contactref element="IC1" pad="9"/>
-<wire x1="57.15" y1="88.9" x2="-54.61" y2="69.85" width="0" layer="19" extent="1-1"/>
+<wire x1="93.98" y1="91.44" x2="-54.61" y2="69.85" width="0" layer="19" extent="1-1"/>
 </signal>
 <signal name="N$5">
 <contactref element="R17" pad="2"/>
 <contactref element="IC1" pad="6"/>
-<wire x1="57.15" y1="81.28" x2="-44.45" y2="69.85" width="0" layer="19" extent="1-1"/>
+<wire x1="93.98" y1="83.82" x2="-44.45" y2="69.85" width="0" layer="19" extent="1-1"/>
 </signal>
 <signal name="AN0">
@@
 <contactref element="IC1" pad="1"/>
 <wire x1="113.03" y1="17.78" x2="-31.75" y2="66.04" width="0" layer="19" extent="1-1"/>
-<wire x1="44.45" y1="81.28" x2="113.03" y2="17.78" width="0" layer="19" extent="1-1"/>
+<wire x1="81.28" y1="83.82" x2="113.03" y2="17.78" width="0" layer="19" extent="1-1"/>
 </signal>
 <signal name="AN1">
@@
 <contactref element="R17" pad="1"/>
 <contactref element="IC1" pad="7"/>
-<wire x1="115.57" y1="17.78" x2="59.69" y2="81.28" width="0" layer="19" extent="1-1"/>
-<wire x1="-52.07" y1="69.85" x2="59.69" y2="81.28" width="0" layer="19" extent="1-1"/>
+<wire x1="115.57" y1="17.78" x2="96.52" y2="83.82" width="0" layer="19" extent="1-1"/>
+<wire x1="-52.07" y1="69.85" x2="96.52" y2="83.82" width="0" layer="19" extent="1-1"/>
 </signal>
 <signal name="AN2">
@@
 <contactref element="R18" pad="1"/>
 <contactref element="IC1" pad="8"/>
-<wire x1="-62.23" y1="69.85" x2="59.69" y2="88.9" width="0" layer="19" extent="1-1"/>
-<wire x1="118.11" y1="17.78" x2="59.69" y2="88.9" width="0" layer="19" extent="1-1"/>
+<wire x1="-62.23" y1="69.85" x2="96.52" y2="91.44" width="0" layer="19" extent="1-1"/>
+<wire x1="118.11" y1="17.78" x2="96.52" y2="91.44" width="0" layer="19" extent="1-1"/>
 </signal>
 <signal name="N$13">

Commit message: Edicion de label conexiones
Connections:
- removed net GND1: R11.A, R9.2
- removed net N$13: ARDUINO_NANO1.12
- new net VIN: ARDUINO_NANO1.15
- net +5V: now also ARDUINO_NANO1.12; no longer ARDUINO_NANO1.15
- net GND: now also R11.A, R9.2
Changed lines of the file:
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@@
 <contactref element="DIS1" pad="5"/>
 <contactref element="220" pad="2"/>
-<wire x1="73.41" y1="73.92" x2="63.25" y2="73.92" width="0" layer="19" extent="1-1"/>
-<wire x1="88.9" y1="91.44" x2="73.41" y2="73.92" width="0" layer="19" extent="1-1"/>
-<wire x1="19.05" y1="43.18" x2="88.9" y2="91.44" width="0" layer="19" extent="1-1"/>
-<wire x1="-36.83" y1="58.42" x2="19.05" y2="43.18" width="0" layer="19" extent="1-1"/>
-<wire x1="-29.21" y1="59.69" x2="-36.83" y2="58.42" width="0" layer="19" extent="1-1"/>
-<wire x1="133.35" y1="33.02" x2="-29.21" y2="59.69" width="0" layer="19" extent="1-1"/>
-<wire x1="-24.13" y1="69.85" x2="-29.21" y2="59.69" width="0" layer="19" extent="1-1"/>
-<wire x1="-13.97" y1="59.69" x2="133.35" y2="33.02" width="0" layer="19" extent="1-1"/>
+<contactref element="R9" pad="2"/>
+<contactref element="R11" pad="A"/>
+<wire x1="73.41" y1="73.92" x2="88.9" y2="91.44" width="0" layer="19" extent="1-1"/>
+<wire x1="63.25" y1="73.92" x2="73.41" y2="73.92" width="0" layer="19" extent="1-1"/>
+<wire x1="15.24" y1="52.07" x2="63.25" y2="73.92" width="0" layer="19" extent="1-1"/>
+<wire x1="19.05" y1="43.18" x2="15.24" y2="52.07" width="0" layer="19" extent="1-1"/>
+<wire x1="-13.97" y1="59.69" x2="15.24" y2="52.07" width="0" layer="19" extent="1-1"/>
+<wire x1="-24.13" y1="69.85" x2="-13.97" y2="59.69" width="0" layer="19" extent="1-1"/>
+<wire x1="-29.21" y1="59.69" x2="-24.13" y2="69.85" width="0" layer="19" extent="1-1"/>
+<wire x1="-36.83" y1="58.42" x2="-29.21" y2="59.69" width="0" layer="19" extent="1-1"/>
+<wire x1="-54.61" y1="66.04" x2="-36.83" y2="58.42" width="0" layer="19" extent="1-1"/>
+<wire x1="133.35" y1="33.02" x2="73.41" y2="73.92" width="0" layer="19" extent="1-1"/>
 <wire x1="138.43" y1="17.78" x2="133.35" y2="33.02" width="0" layer="19" extent="1-1"/>
 </signal>
@@
 <contactref element="R16" pad="E"/>
 <contactref element="IC1" pad="4"/>
-<contactref element="ARDUINO_NANO1" pad="15"/>
 <contactref element="DIS1" pad="2"/>
 <contactref element="DIS1" pad="15"/>
-<wire x1="88.9" y1="83.82" x2="65.79" y2="73.92" width="0" layer="19" extent="1-1"/>
+<contactref element="ARDUINO_NANO1" pad="12"/>
 <wire x1="98.81" y1="73.92" x2="88.9" y2="83.82" width="0" layer="19" extent="1-1"/>
-<wire x1="-34.29" y1="59.69" x2="98.81" y2="73.92" width="0" layer="19" extent="1-1"/>
-<wire x1="-19.05" y1="59.69" x2="-34.29" y2="59.69" width="0" layer="19" extent="1-1"/>
-<wire x1="140.97" y1="17.78" x2="-19.05" y2="59.69" width="0" layer="19" extent="1-1"/>
+<wire x1="65.79" y1="73.92" x2="88.9" y2="83.82" width="0" layer="19" extent="1-1"/>
+<wire x1="133.35" y1="17.78" x2="98.81" y2="73.92" width="0" layer="19" extent="1-1"/>
+<wire x1="-19.05" y1="59.69" x2="65.79" y2="73.92" width="0" layer="19" extent="1-1"/>
+<wire x1="-34.29" y1="59.69" x2="-19.05" y2="59.69" width="0" layer="19" extent="1-1"/>
 </signal>
 <signal name="AC1_3">
@@
 <contactref element="R11" pad="S"/>
 <wire x1="-64.77" y1="66.04" x2="12.7" y2="52.07" width="0" layer="19" extent="1-1"/>
-</signal>
-<signal name="GND1">
-<contactref element="R9" pad="2"/>
-<contactref element="R11" pad="A"/>
-<wire x1="-54.61" y1="66.04" x2="15.24" y2="52.07" width="0" layer="19" extent="1-1"/>
 </signal>
 <signal name="+5V1">
@@
 <wire x1="118.11" y1="17.78" x2="96.52" y2="91.44" width="0" layer="19" extent="1-1"/>
 </signal>
-<signal name="N$13">
-<contactref element="ARDUINO_NANO1" pad="12"/>
-</signal>
 <signal name="D4">
 <contactref element="ARDUINO_NANO1" pad="26"/>
@@
 <wire x1="101.35" y1="73.92" x2="-44.45" y2="58.42" width="0" layer="19" extent="1-1"/>
 </signal>
+<signal name="VIN">
+<contactref element="ARDUINO_NANO1" pad="15"/>
+</signal>
 </signals>

Commit message: primeras ediciones de board
Parts:
- added FASE1: FASE1, con-molex:22-23-2021
- added FASE2: FASE2, con-molex:22-23-2021
- added FASE3: FASE3, con-molex:22-23-2021
- moved R5 119.2 mm to (88.6, 90.9)
- moved R12 104.4 mm to (20.3, 33.0), turned to 180 degrees
- moved 220 97.9 mm to (52.6, 88.3)
- moved R18 97.6 mm to (29.8, 28.1), turned to 270 degrees
- moved R10 91.2 mm to (19.2, 41.5), turned to 180 degrees
- moved R9 86.9 mm to (26.0, 45.3), turned to 90 degrees
- moved R17 80.1 mm to (29.1, 49.2), turned to 90 degrees
- moved R15 74.8 mm to (23.4, 27.3), turned to 270 degrees
- moved IC1 71.9 mm to (36.8, 38.1), turned to 180 degrees
- moved R1 70.7 mm to (19.8, 60.3), turned to 180 degrees
- moved R8 69.9 mm to (19.8, 50.1)
- moved R14 68.4 mm to (26.4, 28.2), turned to 270 degrees
- moved R3 62.5 mm to (40.6, 100.3)
- moved R16 59.7 mm to (17.5, 26.1), turned to 270 degrees
- moved R13 51.3 mm to (20.3, 35.6)
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Connections:
- net AC1_1: now also FASE1.1
- net AC1_2: now also FASE1.2
- net AC1_3: now also FASE2.1
- net AC1_4: now also FASE2.2
- net AC1_5: now also FASE3.1
- net AC1_6: now also FASE3.2
Routing:
- net GND: track 0.00 -> 31.6 mm
- net IN2: track 0.00 -> 24.2 mm
- net IN3: track 0.00 -> 21.6 mm
- net N$5: track 0.00 -> 12.2 mm
- net N$1: track 0.00 -> 11.4 mm
- net OFFSET3: track 0.00 -> 8.02 mm
- net IN1: track 0.00 -> 6.57 mm
- net AC1_1: track 0.00 -> 5.10 mm
- net AC1_6: track 0.00 -> 5.08 mm
- net AC1_5: track 0.00 -> 5.08 mm
- net AC1_4: track 0.00 -> 5.08 mm
- net AC1_3: track 0.00 -> 5.08 mm
- net AC1_2: track 0.00 -> 5.08 mm
- net OFFSET1: track 0.00 -> 4.86 mm
- net OFFSET2: track 0.00 -> 3.81 mm
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
Commit message: Ruteo sin union con arduino
Parts:
- moved R5 62.8 mm to (41.8, 49.1), turned to 270 degrees
- moved R3 43.7 mm to (26.2, 59.1), turned to 270 degrees
- moved 220 37.7 mm to (28.8, 59.0), turned to 270 degrees
Connections:
- removed net +5V1: R11.E
- net +5V: now also R11.E
Routing:
- net +5V: track 0.00 -> 60.7 mm
- net GND: track 31.6 -> 79.0 mm
- net IN1: track 6.57 -> 36.8 mm
- net AN0: track 0.00 -> 12.0 mm
- net N$2: track 0.00 -> 3.37 mm
- net IN3: track 21.6 -> 20.3 mm
- net IN2: track 24.2 -> 23.2 mm
