File: PCB´s/VoltimetroTrifasico/sch2.sch (EAGLE design)
At the start: 25 parts, among them IC1 LM324N

Commit message: Rutas con Arduino y se agrego mol para fuente
Parts:
- removed DIS1: TUXGR_16X2_R2, display-lcd:TUXGR_16X2_R2
- added FTE: FTE, con-molex:22-23-2021
- added R19: (no value), pot:TRIM_EU-B64Y
- added X1: LCD1, con-molex:22-23-2061
- added X3: LCD2, con-molex:22-23-2061
Connections:
- removed net N$3: 220.1, DIS1.NC@2
- new net RES: 220.1, X3-6.S
- net +5V: now also FTE-1.S, R19.E, X1-2.S, X3-5.S; no longer DIS1.NC@1, DIS1.VCC
- net D4: now also X3-1.S; no longer DIS1.D4
- net D5: now also X3-2.S; no longer DIS1.D5
- net D6: now also X3-3.S; no longer DIS1.D6
- net D7: now also X3-4.S; no longer DIS1.D7
- net ENA: now also X1-6.S; no longer DIS1.E
- net GND: now also FTE-2.S, R19.A, X1-1.S, X1-5.S; no longer DIS1.GND, DIS1.R/W
- net RS: now also X1-4.S; no longer DIS1.RS
- net V0: now also R19.S, X1-3.S; no longer DIS1.CONTR
Other:
- moved on the sheet: 220
Changed lines of the file:
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@@
 <part name="R18" library="rcl" deviceset="R-US_" device="0204/7" value="10k"/>
 <part name="ARDUINO_NANO1" library="ArduinoNanoV30" deviceset="ARDUINO_NANO" device=""/>
-<part name="DIS1" library="display-lcd" deviceset="TUXGR_16X2_R2" device=""/>
 <part name="220" library="rcl" deviceset="R-US_" device="0204/7" value="10k"/>
 <part name="FASE1" library="con-molex" deviceset="22-23-2021" device="" value="FASE1"/>
 <part name="FASE2" library="con-molex" deviceset="22-23-2021" device="" value="FASE2"/>
 <part name="FASE3" library="con-molex" deviceset="22-23-2021" device="" value="FASE3"/>
+<part name="FTE" library="con-molex" deviceset="22-23-2021" device="" value="FTE"/>
+<part name="R19" library="pot" deviceset="TRIM_EU-" device="B64Y"/>
+<part name="X1" library="con-molex" deviceset="22-23-2061" device="" value="LCD1"/>
+<part name="X3" library="con-molex" deviceset="22-23-2061" device="" value="LCD2"/>
 </parts>
 <sheets>
@@
 <instance part="IC1" gate="P" x="48.26" y="104.14"/>
 <instance part="ARDUINO_NANO1" gate="G$1" x="91.44" y="76.2"/>
-<instance part="DIS1" gate="G$1" x="139.7" y="83.82" rot="R270"/>
-<instance part="220" gate="G$1" x="121.92" y="63.5" rot="R180"/>
+<instance part="220" gate="G$1" x="99.06" y="10.16" rot="R180"/>
 <instance part="FASE1" gate="-1" x="17.78" y="0" rot="R180"/>
 <instance part="FASE1" gate="-2" x="17.78" y="2.54" rot="R180"/>
@@
 <instance part="FASE3" gate="-1" x="17.78" y="25.4" rot="R180"/>
 <instance part="FASE3" gate="-2" x="17.78" y="27.94" rot="R180"/>
+<instance part="FTE" gate="-1" x="33.02" y="15.24"/>
+<instance part="FTE" gate="-2" x="33.02" y="12.7"/>
+<instance part="R19" gate="1" x="106.68" y="35.56"/>
+<instance part="X1" gate="-1" x="121.92" y="43.18"/>
+<instance part="X1" gate="-2" x="121.92" y="40.64"/>
+<instance part="X1" gate="-3" x="121.92" y="38.1"/>
+<instance part="X1" gate="-4" x="121.92" y="35.56"/>
+<instance part="X1" gate="-5" x="121.92" y="33.02"/>
+<instance part="X1" gate="-6" x="121.92" y="30.48"/>
+<instance part="X3" gate="-1" x="121.92" y="22.86"/>
+<instance part="X3" gate="-2" x="121.92" y="20.32"/>
+<instance part="X3" gate="-3" x="121.92" y="17.78"/>
+<instance part="X3" gate="-4" x="121.92" y="15.24"/>
+<instance part="X3" gate="-5" x="121.92" y="12.7"/>
+<instance part="X3" gate="-6" x="121.92" y="10.16"/>
 </instances>
 <busses>
@@
 </segment>
 <segment>
-<pinref part="DIS1" gate="G$1" pin="GND"/>
-<junction x="129.54" y="101.6"/>
-<label x="129.54" y="101.6" size="1.778" layer="95" rot="R180"/>
-</segment>
-<segment>
-<pinref part="DIS1" gate="G$1" pin="R/W"/>
-<junction x="129.54" y="91.44"/>
-<label x="129.54" y="91.44" size="1.778" layer="95" rot="R180"/>
-</segment>
-<segment>
 <pinref part="220" gate="G$1" pin="2"/>
-<junction x="116.84" y="63.5"/>
-<label x="116.84" y="63.5" size="1.778" layer="95" rot="R180"/>
+<junction x="93.98" y="10.16"/>
+<label x="93.98" y="10.16" size="1.778" layer="95" rot="R180"/>
 </segment>
 <segment>
@@
 <label x="-15.24" y="71.12" size="1.778" layer="95"/>
 </segment>
+<segment>
+<pinref part="FTE" gate="-2" pin="S"/>
+<junction x="30.48" y="12.7"/>
+</segment>
+<segment>
+<pinref part="R19" gate="1" pin="A"/>
+<junction x="106.68" y="30.48"/>
+</segment>
+<segment>
+<pinref part="X1" gate="-1" pin="S"/>
+<junction x="119.38" y="43.18"/>
+<label x="111.76" y="43.18" size="1.778" layer="95"/>
+</segment>
+<segment>
+<pinref part="X1" gate="-5" pin="S"/>
+<junction x="119.38" y="33.02"/>
+<label x="114.3" y="33.02" size="1.778" layer="95"/>
+</segment>
 </net>
 <net name="+5V" class="0">
@@
 </segment>
 <segment>
-<pinref part="DIS1" gate="G$1" pin="VCC"/>
-<junction x="129.54" y="99.06"/>
-<label x="129.54" y="99.06" size="1.778" layer="95" rot="R180"/>
-</segment>
-<segment>
-<pinref part="DIS1" gate="G$1" pin="NC@1"/>
-<junction x="129.54" y="66.04"/>
-<label x="129.54" y="66.04" size="1.778" layer="95" rot="R180"/>
-</segment>
-<segment>
 <pinref part="ARDUINO_NANO1" gate="G$1" pin="5V"/>
 <junction x="111.76" y="91.44"/>
@@
 <junction x="-7.62" y="83.82"/>
 <label x="-7.62" y="86.36" size="1.778" layer="95"/>
+</segment>
+<segment>
+<pinref part="FTE" gate="-1" pin="S"/>
+<junction x="30.48" y="15.24"/>
+</segment>
+<segment>
+<pinref part="R19" gate="1" pin="E"/>
+<junction x="106.68" y="40.64"/>
+</segment>
+<segment>
+<pinref part="X1" gate="-2" pin="S"/>
+<junction x="119.38" y="40.64"/>
+<label x="111.76" y="40.64" size="1.778" layer="95"/>
+</segment>
+<segment>
+<pinref part="X3" gate="-5" pin="S"/>
+<junction x="119.38" y="12.7"/>
+<label x="114.3" y="12.7" size="1.778" layer="95"/>
 </segment>
 </net>
@@
 </segment>
 <segment>
-<pinref part="DIS1" gate="G$1" pin="D4"/>
-<junction x="129.54" y="76.2"/>
-<label x="129.54" y="76.2" size="1.778" layer="95" rot="R180"/>
+<pinref part="X3" gate="-1" pin="S"/>
+<junction x="119.38" y="22.86"/>
+<label x="114.3" y="22.86" size="1.778" layer="95"/>
 </segment>
 </net>
@@
 </segment>
 <segment>
-<pinref part="DIS1" gate="G$1" pin="D7"/>
-<junction x="129.54" y="68.58"/>
-<label x="129.54" y="68.58" size="1.778" layer="95" rot="R180"/>
+<pinref part="X3" gate="-4" pin="S"/>
+<junction x="119.38" y="15.24"/>
+<label x="114.3" y="15.24" size="1.778" layer="95"/>
 </segment>
 </net>
@@
 </segment>
 <segment>
-<pinref part="DIS1" gate="G$1" pin="D6"/>
-<junction x="129.54" y="71.12"/>
-<label x="129.54" y="71.12" size="1.778" layer="95" rot="R180"/>
+<pinref part="X3" gate="-3" pin="S"/>
+<junction x="119.38" y="17.78"/>
+<label x="114.3" y="17.78" size="1.778" layer="95"/>
 </segment>
 </net>
@@
 </segment>
 <segment>
-<pinref part="DIS1" gate="G$1" pin="D5"/>
-<junction x="129.54" y="73.66"/>
-<label x="129.54" y="73.66" size="1.778" layer="95" rot="R180"/>
+<pinref part="X3" gate="-2" pin="S"/>
+<junction x="119.38" y="20.32"/>
+<label x="114.3" y="20.32" size="1.778" layer="95"/>
 </segment>
 </net>
@@
 </segment>
 <segment>
-<pinref part="DIS1" gate="G$1" pin="E"/>
-<junction x="129.54" y="88.9"/>
-<label x="129.54" y="88.9" size="1.778" layer="95" rot="R180"/>
+<pinref part="X1" gate="-6" pin="S"/>
+<junction x="119.38" y="30.48"/>
+<label x="111.76" y="30.48" size="1.778" layer="95"/>
 </segment>
 </net>
@@
 </segment>
 <segment>
-<pinref part="DIS1" gate="G$1" pin="RS"/>
-<junction x="129.54" y="93.98"/>
-<label x="129.54" y="93.98" size="1.778" layer="95" rot="R180"/>
+<pinref part="X1" gate="-4" pin="S"/>
+<junction x="119.38" y="35.56"/>
+<label x="114.3" y="35.56" size="1.778" layer="95"/>
 </segment>
 </net>
 <net name="V0" class="0">
 <segment>
-<pinref part="DIS1" gate="G$1" pin="CONTR"/>
-<junction x="129.54" y="96.52"/>
-<label x="129.54" y="96.52" size="1.778" layer="95" rot="R180"/>
-</segment>
-</net>
-<net name="N$3" class="0">
-<segment>
-<pinref part="DIS1" gate="G$1" pin="NC@2"/>
+<pinref part="R19" gate="1" pin="S"/>
+<junction x="111.76" y="35.56"/>
+<label x="111.76" y="33.02" size="1.778" layer="95"/>
+</segment>
+<segment>
+<pinref part="X1" gate="-3" pin="S"/>
+<junction x="119.38" y="38.1"/>
+<label x="111.76" y="38.1" size="1.778" layer="95"/>
+</segment>
+</net>
+<net name="RES" class="0">
+<segment>
+<pinref part="X3" gate="-6" pin="S"/>
+<junction x="119.38" y="10.16"/>
+<label x="114.3" y="10.16" size="1.778" layer="95"/>
+</segment>
+<segment>
 <pinref part="220" gate="G$1" pin="1"/>
-<wire x1="129.54" y1="63.5" x2="127" y2="63.5" width="0.1524" layer="91"/>
-</segment>
-</net>
+<wire x1="106.68" y1="10.16" x2="104.14" y2="10.16" width="0.1524" layer="91"/>
+<junction x="106.68" y="10.16"/>
+<label x="106.68" y="10.16" size="1.778" layer="95"/>
+</segment>
+</net>

Commit message: ruteo terminado
Connections:
- net AN0: now also IC1B.OUT, R17.1; no longer IC1A.OUT, R5.1
- net AN1: now also IC1A.OUT, R5.1; no longer IC1B.OUT, R17.1
Changed lines of the file:
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@@
-</segment>
-<segment>
-<pinref part="R5" gate="G$1" pin="1"/>
-<pinref part="IC1" gate="A" pin="OUT"/>
-<wire x1="43.18" y1="96.52" x2="43.18" y2="104.14" width="0.1524" layer="91"/>
-<junction x="43.18" y="104.14"/>
-<label x="48.26" y="104.14" size="1.778" layer="95" rot="R180"/>
-</segment>
-</net>
-<net name="AN1" class="0">
-<segment>
-<pinref part="ARDUINO_NANO1" gate="G$1" pin="ADC1/A1"/>
-<junction x="111.76" y="73.66"/>
 </segment>
 <segment>
@@
 </segment>
 </net>
+<net name="AN1" class="0">
+<segment>
+<pinref part="ARDUINO_NANO1" gate="G$1" pin="ADC1/A1"/>
+<junction x="111.76" y="73.66"/>
+</segment>
+<segment>
+<pinref part="R5" gate="G$1" pin="1"/>
+<pinref part="IC1" gate="A" pin="OUT"/>
+<wire x1="43.18" y1="96.52" x2="43.18" y2="104.14" width="0.1524" layer="91"/>
+<junction x="43.18" y="104.14"/>
+<label x="48.26" y="104.14" size="1.778" layer="95" rot="R180"/>
+</segment>
+</net>
